File: Relay_RS485.kicad_sch (KiCad schematic)
At the start: 86 parts, among them J1 RELAY_CONN, J2 SWD, J4 RS485_POWER, Q1 NPN, Q2 NPN, Q3 NPN, Q4 NPN, SW1 reset, U1 XL1509, U2 MAX3485, U3 STM32F030F4Px, U4 RT9193-33, U5 LM358

Commit message: Finish board.
Parts:
- removed H1: ACO, symbol Mechanical:MountingHole_Pad
- removed H2: ACI, symbol Mechanical:MountingHole_Pad
- removed J1: RELAY_CONN, symbol Connector:Screw_Terminal_01x06
- removed U2: MAX3485, symbol Interface_UART:MAX3485
- added C19, C20: 100nF, Anh_Footprints:C_0603, symbol Device:C_Small
- added H3: H1, MountingHole:MountingHole_3.2mm_M3_Pad_Via, symbol Mechanical:MountingHole_Pad
- added H4: ACO, MountingHole:MountingHole_3.2mm_M3_Pad_Via, symbol Mechanical:MountingHole_Pad
- added H5: H3, MountingHole:MountingHole_3.2mm_M3_Pad_Via, symbol Mechanical:MountingHole_Pad
- added H6: H4, MountingHole:MountingHole_3.2mm_M3_Pad_Via, symbol Mechanical:MountingHole_Pad
- added J1: OUTPUT_CONN, TerminalBlock_Phoenix:TerminalBlock_Phoenix_MKDS-1,5-8-5.08_1x08_P5.08mm_Horizontal, symbol Connector:Screw_Terminal_01x08
- added U2: MAX485E, Anh_Footprints:SOIC-8, symbol Interface_UART:MAX485E
- C1, C10, C12, C14, C15, C17, C18, C2, C3, C5, C8, C9: footprint (none) -> Anh_Footprints:C_0603
- C11, C13, C16, C4, C6: footprint (none) -> Anh_Footprints:C_1210
- C7: footprint (none) -> Capacitor_SMD:CP_Elec_6.3x5.4_Nichicon
- D11, D13, D6, D7, D9: footprint (none) -> Anh_Footprints:LED_0603
- D14: footprint Diode_SMD:D_MiniMELF -> Anh_Footprints:D_MiniMELF
- F1, F2: footprint (none) -> Anh_Footprints:F_1812
- J2: footprint (none) -> Connector_PinHeader_2.54mm:PinHeader_1x04_P2.54mm_Vertical
- J4: footprint (none) -> TerminalBlock_Phoenix:TerminalBlock_Phoenix_MKDS-1,5-8-5.08_1x08_P5.08mm_Horizontal
- R1, R10, R11, R12, R13, R14, R15, R16, R17, R18, R19, R2, R20, R21, R22, R23, R24, R25, R26, R27, R28, R3, R4, R5, R6, R7, R8: footprint (none) -> Anh_Footprints:R_0603
- R9: footprint (none) -> Anh_Footprints:R_0805
- RL1, RL2, RL3, RL4: footprint IVSfootprint:G5NB-1A-E DC5 -> IVS_Footprint:Relay_G5NB-1A-E DC5
- RV1, RV2: footprint (none) -> Potentiometer_SMD:Potentiometer_Bourns_3314J_Vertical
- SW1: footprint (none) -> Button_Switch_SMD:SW_SPST_CK_RS282G05A3
- U5: footprint (none) -> Anh_Footprints:SOIC-8
Connections:
- net +3V3: now also C19.2, C20.2; no longer C2.2, R3.2, R8.2
- net +5V: now also C2.2, R3.2, R8.2, U1.3 (FB), U2.8 (VCC)
- net A+: now also J4.3 (Pin_3), J4.4 (Pin_4); no longer J4.7 (Pin_7), J4.8 (Pin_8)
- net B-: now also J4.7 (Pin_7), J4.8 (Pin_8); no longer J4.3 (Pin_3), J4.4 (Pin_4)
- net COM: now also RL1.2, RL2.2, RL3.2, RL4.2, J1.3 (Pin_3), J1.6 (Pin_6); no longer CT1.3 (AC1), RL1.3, RL2.3, RL3.3, RL4.3
- net GND: now also J4.1 (Pin_1), RV2.1, C19.1, C20.1, J1.1 (Pin_1), U2.5 (GND); no longer J4.2 (Pin_2), RV2.3
- net RL1: now also RL1.3, J1.4 (Pin_4); no longer RL1.2
- net RL2: now also RL2.3, J1.5 (Pin_5); no longer RL2.2
- net RL3: now also RL3.3, J1.7 (Pin_7); no longer RL3.2
- net RL4: now also RL4.3, J1.8 (Pin_8); no longer RL4.2
- net VCC: now also J4.2 (Pin_2); no longer J4.1 (Pin_1)
- net at D1.2 (A2), D2.1 (A1), F2.1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: now also U2.6 (A)
- net at D2.2 (A2), D3.1 (A1), F1.1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: now also U2.7 (B)
- net at D15.1: now also RV2.3; no longer RV2.1
- net at R5.2, R8.1: now also U2.1 (RO)
- net at R6.2: now also U2.2 (~{RE}), U2.3 (DE)
- net at R7.2: now also U2.4 (DI)
- net at U5.1, U5.5 (+): now also RV1.3; no longer RV1.1
- net at R27.2, RV1.2: now also RV1.1; no longer RV1.3
- net S+: now reaches C16.2, CT1.2 (O2)
- net S+: now also J1.2 (Pin_2)
- removed net COM_C: CT1.4 (AC2)
- no-connect marks 4 -> 8
Other:
- moved on the sheet: J4, RV1
